File: KiCAD/ardPWMFan/ardPWMFan.kicad_pcb (KiCad board)
At the start: 2 copper layers, 78.7 x 51.4 mm, 19 parts, among them J1 Conn_01x02, M1 Fan, Q1 20N6003, U1 DS18B20, U2 2-pole_power_in_screw_terminal, U3 Arduino_Mini_Pro, U4 TM1637_4x7-segment_display, U5 L7805

Commit message: working...
Routing:
- net GND: track 188.3 -> 180.0 mm
- net Net-(M1-Pad2): track 76.2 -> 77.7 mm
Other:
- board text added: "D3"

Commit message: kicad6
Routing:
- net +5V: track 215.8 -> 212.7 mm
- net GND: track 180.0 -> 181.4 mm
- net Net-(R2-Pad2): track 53.7 -> 52.5 mm
- net +12Vf: track 54.7 -> 53.6 mm
- net Net-(C4-Pad1): track 14.5 -> 13.4 mm
- net Net-(M1-Pad2): track 77.7 -> 76.9 mm
- net Net-(J1-Pad2): track 28.5 -> 27.8 mm
Other:
- net class 30 removed
- net class Default removed
